File: dick_mouse_circuit/_restore_backup_2026-09-09T20-42-40-775/dick_mouse.kicad_sch (KiCad schematic)
At the start: 52 parts, among them J1 USB_C_Receptacle_USB2.0_16P, J10 Conn_01x04, J11 Conn_01x09, J2 AudioJack3, J3 Conn_01x03, J4 Conn_01x03, J5 Conn_01x03, J6 Conn_01x02, J7 Conn_01x02, J8 Conn_01x05, J9 Conn_01x05, SW1 SW_Push, SW2 SW_Push, SW3 SW_Push, SW4 SW_Push, SW5 SW_Push, SW6 SW_Push, SW7 SW_Wuerth_450301014042, U1 USBLC6-2SC6, U2 ESP32-S3-WROOM-1, U3 AMS1117-3.3, U4 PCM5102A

Commit message: マイク調整済み
Parts:
- removed C13, C14, C15, C17: 10u, Capacitor_SMD:C_0603_1608Metric, symbol Device:C
- removed SW7: SW_Wuerth_450301014042, Button_Switch_THT:SW_Slide-03_Wuerth-WS-SLTV_10x2.5x6.4_P2.54mm, symbol Switch:SW_Wuerth_450301014042
- added C13, C14, C15, C17: 10u, symbol Device:C_Polarized
- added SW7: SW_Push, symbol Switch:SW_Push
- C1, C10, C11, C12, C16, C3, C6, C7, C8, C9: footprint Capacitor_SMD:C_0402_1005Metric -> (none)
- C2, C4, C5: footprint Capacitor_SMD:CP_Elec_5x5.9 -> (none)
- D1, D2: footprint LED_SMD:LED_0603_1608Metric -> (none)
- D3: renamed from D4; footprint LED_SMD:LED_0603_1608Metric -> (none)
- J10: footprint Connector_PinHeader_2.54mm:PinHeader_1x04_P2.54mm_Vertical -> (none)
- J11: footprint Connector_PinHeader_2.54mm:PinHeader_1x09_P2.54mm_Vertical -> (none)
- J3, J4, J5: footprint Connector_PinHeader_2.54mm:PinHeader_1x03_P2.54mm_Vertical -> (none)
- J6, J7: footprint Connector_PinHeader_2.54mm:PinHeader_1x02_P2.54mm_Vertical -> (none)
- J8, J9: footprint Connector_PinHeader_2.54mm:PinHeader_1x05_P2.54mm_Vertical -> (none)
- R1, R2, R3, R4, R5, R6, R7, R8: footprint Resistor_SMD:R_0402_1005Metric -> (none)
- SW1, SW2, SW3, SW4, SW5, SW6: footprint Button_Switch_SMD:SW_Push_1P1T_NO_CK_KSC6xxG -> (none)
- renumbered D3 to D4, U3 to U4, U4 to U5
Connections:
- net +5V: now also C13.1, C15.1, C17.1
- net GND: now also C14.2, C15.2, C17.2, SW7.2
- net LDOO: now also C13.2, C14.1
- net SW7: now also SW7.1
- no-connect marks 3 -> 2
Other:
- company: 株式会社ウメモドキ -> (none)
- title: おちんちんマウス回路 -> (none)
