File: dick_mouse_circuit/dick_mouse.kicad_sch (KiCad schematic)
At the start: 52 parts, among them J1 USB_C_Receptacle_USB2.0_16P, J10 Conn_01x04, J11 Conn_01x09, J2 AudioJack3, J3 Conn_01x03, J4 Conn_01x03, J5 Conn_01x03, J6 Conn_01x02, J7 Conn_01x02, J8 Conn_01x05, J9 Conn_01x05, SW1 SW_Push, SW2 SW_Push, SW3 SW_Push, SW4 SW_Push, SW5 SW_Push, SW6 SW_Push, SW7 SW_Wuerth_450301014042, U1 USBLC6-2SC6, U2 ESP32-S3-WROOM-1, U3 AMS1117-3.3, U4 PCM5102A

Commit message: pcb編集中
Parts:
- removed D1, D2: LED, LED_SMD:LED_0603_1608Metric, symbol Device:LED
- removed R2, R3: 470, Resistor_SMD:R_0402_1005Metric, symbol Device:R
- C1, C10, C11, C16, C3, C9: LCSC (none) -> C1525; MPN (none) -> CL05B104KO5NNNC; Manufacturer (none) -> Samsung Electro-Mechanics
- C12, C6: LCSC (none) -> C12530; MPN (none) -> CL05A225MQ5NSNC; Manufacturer (none) -> Samsung Electro-Mechanics
- C13, C14, C15, C17: LCSC (none) -> C96446; MPN (none) -> CL10A106MA8NRNC; Manufacturer (none) -> Samsung Electro-Mechanics
- C2, C5: footprint Capacitor_SMD:CP_Elec_5x5.9 -> Capacitor_SMD:C_0805_2012Metric; symbol Device:C_Polarized -> Device:C; LCSC (none) -> C45783; MPN (none) -> CL21A226MAQNNNE; Manufacturer (none) -> Samsung Electro-Mechanics
- C4: footprint Capacitor_SMD:CP_Elec_5x5.9 -> Capacitor_SMD:C_0603_1608Metric; symbol Device:C_Polarized -> Device:C; LCSC (none) -> C96446; MPN (none) -> CL10A106MA8NRNC; Manufacturer (none) -> Samsung Electro-Mechanics
- C7, C8: LCSC (none) -> C1531; MPN (none) -> 0402B222K500NT; Manufacturer (none) -> FH
- D3, D5: LCSC (none) -> C8678; MPN (none) -> SS34; Manufacturer (none) -> MDD(Microdiode Semiconductor)
- D4: value LED -> Red LED; LCSC (none) -> C2286; MPN (none) -> KT-0603R; Manufacturer (none) -> Hubei KENTO Elec
- J1: value USB_C_Receptacle_USB2.0_16P -> TYPE-C-31-M-12; footprint Connector_USB:USB_C_Receptacle_Amphenol_12401948E412A -> Connector_USB:USB_C_Receptacle_HRO_TYPE-C-31-M-12; LCSC (none) -> C165948; MPN (none) -> TYPE-C-31-M-12; Manufacturer (none) -> Korean Hroparts Elec
- J10: LCSC (none) -> C2691448; MPN (none) -> PZ254V-11-04P; Manufacturer (none) -> XFCN
- J11: LCSC (none) -> C492408; MPN (none) -> PZ254V-11-09P; Manufacturer (none) -> XFCN
- J2: BOM Notes (none) -> LCSC candidate only; keep current CUI SJ-3523 footprint unt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; LCSC (none) -> C668608; MPN (none) -> PJ-313D; Manufacturer (none) -> SHOU HAN
- J3, J4, J5: LCSC (none) -> C2937625; MPN (none) -> PZ254V-11-03P; Manufacturer (none) -> XFCN
- J6, J7: LCSC (none) -> C492401; MPN (none) -> PZ254V-11-02P; Manufacturer (none) -> XFCN
- J8, J9: LCSC (none) -> C492404; MPN (none) -> PZ254V-11-05P; Manufacturer (none) -> XFCN
- R1: LCSC (none) -> C25744; MPN (none) -> 0402WGF1002TCE; Manufacturer (none) -> UNI-ROYAL
- R4, R5: LCSC (none) -> C25905; MPN (none) -> 0402WGF5101TCE; Manufacturer (none) -> UNI-ROYAL
- R6, R7, R8: LCSC (none) -> C25117; MPN (none) -> 0402WGF4700TCE; Manufacturer (none) -> UNI-ROYAL
- SW1, SW2, SW3, SW4, SW5, SW6: value SW_Push -> TS-1187A-B-A-B; footprint Button_Switch_SMD:SW_Push_1P1T_NO_CK_KSC6xxG -> Button_Switch_SMD:SW_Push_1P1T_XKB_TS-1187A; LCSC (none) -> C318884; MPN (none) -> TS-1187A-B-A-B; Manufacturer (none) -> XKB Connection
- SW7: value SW_Wuerth_450301014042 -> SS-12D00-G3; BOM Notes (none) -> LCSC candidate only; current Wuerth footprint kept because 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; LCSC (none) -> C22355741; MPN (none) -> SS-12D00-G3; Manufacturer (none) -> SOFNG
- U3: LCSC (none) -> C6186; MPN (none) -> AMS1117-3.3; Manufacturer (none) -> Advanced Monolithic Systems
Connections:
- net +3.3V: now also C11.1, C13.1, C15.1, C16.1, C17.1, C9.1, U4.1 (CPVDD), U4.17 (XSMT), U4.20 (DVDD), U4.8 (AVDD); no longer J11.8 (Pin_8)
- net +5V: no longer C11.1, C13.1, C15.1, C16.1, C17.1, C9.1, U4.1 (CPVDD), U4.17 (XSMT), U4.20 (DVDD), U4.8 (AVDD)
- net GND: no longer J11.9 (Pin_9)
- net IO45: now also J11.8 (Pin_8)
- net IO46: now also J11.9 (Pin_9)

Commit message: 基板完成
Parts:
- removed J11: Conn_01x09, Connector_PinHeader_2.54mm:PinHeader_1x09_P2.54mm_Vertical, symbol Connector_Generic:Conn_01x09
- removed J3, J4: Conn_01x03, Connector_PinHeader_2.54mm:PinHeader_1x03_P2.54mm_Vertical, symbol Connector_Generic:Conn_01x03
- removed SW5, SW6: TS-1187A-B-A-B, Button_Switch_SMD:SW_Push_1P1T_XKB_TS-1187A, symbol Switch:SW_Push
- removed SW7: SS-12D00-G3, Button_Switch_THT:SW_Slide-03_Wuerth-WS-SLTV_10x2.5x6.4_P2.54mm, symbol Switch:SW_Wuerth_450301014042
- added H1, H2, H3, H4: MountingHole, MountingHole:MountingHole_3.2mm_M3, symbol Mechanical:MountingHole
- added J11, J13: Conn_01x04, Connector_PinHeader_2.54mm:PinHeader_1x04_P2.54mm_Vertical, symbol Connector_Generic:Conn_01x04
- added J12: Conn_01x02, Connector_JST:JST_XH_B2B-XH-A_1x02_P2.50mm_Vertical, symbol Connector_Generic:Conn_01x02
- added J3, J4: Conn_01x05, Connector_JST:JST_XH_B5B-XH-A_1x05_P2.50mm_Vertical, symbol Connector_Generic:Conn_01x05
- J2: footprint Connector_Audio:Jack_3.5mm_CUI_SJ-3523-SMT_Horizontal -> lcsc_footprints:C668608_PJ-313D; BOM Notes LCSC candidate only; keep current CUI SJ-3523 footprint unt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 -> Uses the project-local C668608_PJ-313D footprint and 3D mod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
- J5: footprint Connector_PinHeader_2.54mm:PinHeader_1x03_P2.54mm_Vertical -> Connector_JST:JST_XH_B3B-XH-A_1x03_P2.50mm_Vertical
- J6, J7: footprint Connector_PinHeader_2.54mm:PinHeader_1x02_P2.54mm_Vertical -> Connector_JST:JST_XH_B2B-XH-A_1x02_P2.50mm_Vertical
- J8, J9: footprint Connector_PinHeader_2.54mm:PinHeader_1x05_P2.54mm_Vertical -> Connector_JST:JST_XH_B5B-XH-A_1x05_P2.50mm_Vertical
- renumbered D3 to D1, D4 to D2, D5 to D3, R4 to R2, R5 to R3, R6 to R4, R7 to R5, R8 to R6
Connections:
- net SW5 is gone; now on net SW_LEFT: U2.33 (IO40)
- net SW6 is gone; now on net SW_RIGHT: U2.34 (IO41)
- net +3.3V: now also J3.1 (Pin_1), J4.1 (Pin_1)
- net BCLK_TX: now also U2.10 (IO17); no longer U2.8 (IO15)
- net GND: now also J12.2 (Pin_2), J3.5 (Pin_5), J4.5 (Pin_5)
- net IO18: now also J11.2 (Pin_2)
- net IO3: now also J11.3 (Pin_3)
- net IO35: now also J13.3 (Pin_3)
- net IO36: now also J13.2 (Pin_2)
- net IO37: now also J13.1 (Pin_1)
- net IO4: now also J11.1 (Pin_1)
- net IO45: now also J13.4 (Pin_4)
- net IO46: now also J11.4 (Pin_4)
- net SD_TX: now also U2.9 (IO16); no longer U2.10 (IO17)
- net SW_LEFT: now also SW3.1; no longer J6.1 (Pin_1), U2.24 (IO47)
- net SW_RIGHT: now also SW4.1; no longer J7.1 (Pin_1), U2.25 (IO48)
- net WS_TX: now also U2.8 (IO15); no longer U2.9 (IO16)
- net ENC1_A renamed ENC_A_MIC
- net ENC_A_MIC: now also J3.4 (Pin_4)
- net ENC1_B renamed ENC_B_MIC
- net ENC_B_MIC: now also J3.3 (Pin_3)
- net ENC2_A renamed SW_MIC
- net SW_MIC: now also J3.2 (Pin_2)
- net ENC2_B renamed ENC_A_SPK
- net ENC_A_SPK: now also J4.4 (Pin_4)
- net ENC3_A renamed ENC_B_MOUSE
- net ENC_B_MOUSE: now also U2.32 (IO39); no longer U2.21 (IO13)
- net ENC3_B renamed ENC_A_MOUSE
- net ENC_A_MOUSE: now also U2.31 (IO38); no longer U2.22 (IO14)
- removed net SW3: SW3.1, U2.31 (IO38)
- removed net SW4: SW4.1, U2.32 (IO39)
- net SW7 renamed SW_SWAP
- net SW_SWAP: now also J12.1 (Pin_1)
- new net ENC_B_SPK: J4.3 (Pin_3), U2.21 (IO13)
- new net SW_BACK: J7.1 (Pin_1), U2.25 (IO48)
- new net SW_FORWARD: J6.1 (Pin_1), U2.24 (IO47)
- new net SW_SPK: J4.2 (Pin_2), U2.22 (IO14)
- no-connect marks 3 -> 2

Commit message: 基板発注前更新
Parts:
- SW3, SW4: value TS-1187A-B-A-B -> Tactile Switch 6x6x6mm THT; footprint Button_Switch_SMD:SW_Push_1P1T_XKB_TS-1187A -> Button_Switch_THT:SW_PUSH_6mm; BOM Comments (none) -> Amazon ASIN B084XBRQVN; verify 6.5x4.5 mm pin spacing befor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; LCSC C318884 -> (none); MPN TS-1187A-B-A-B -> (none); Manufacturer XKB Connection -> Generic
Connections:
- net +3.3V: now also J9.1 (Pin_1); no longer J9.4 (Pin_4)
- net BCLK_RX: now also J9.3 (Pin_3); no longer J9.1 (Pin_1)
- net GND: now also J9.2 (Pin_2); no longer J9.5 (Pin_5)
- net IO3: now also J11.4 (Pin_4); no longer J11.3 (Pin_3)
- net IO46: now also J11.3 (Pin_3); no longer J11.4 (Pin_4)
- net SD_RX: now also J9.5 (Pin_5); no longer J9.3 (Pin_3)
- net USB_DM: now also U1.6 (I/O1); no longer U1.1 (I/O1)
- net USB_DP: now also U1.4 (I/O2); no longer U1.3 (I/O2)
- net WS_RX: now also J9.4 (Pin_4); no longer J9.2 (Pin_2)
- net at J1.A6 (D+), J1.B6 (D+): now also U1.3 (I/O2); no longer U1.4 (I/O2)
- net at J1.A7 (D-), J1.B7 (D-): now also U1.1 (I/O1); no longer U1.6 (I/O1)
