File: dick_mouse_circuit/dick_mouse.kicad_pcb (KiCad board)
At the start: 2 copper layers, 4.5 x 13.4 mm, 52 parts, among them J1 USB_C_Receptacle_USB2.0_16P, J10 Conn_01x04, J11 Conn_01x09, J2 AudioJack3, J3 Conn_01x03, J4 Conn_01x03, J5 Conn_01x03, J6 Conn_01x02, J7 Conn_01x02, J8 Conn_01x05, J9 Conn_01x05, SW1 SW_Push, SW2 SW_Push, SW3 SW_Push, SW4 SW_Push, SW5 SW_Push, SW6 SW_Push, SW7 SW_Wuerth_450301014042, U1 USBLC6-2SC6, U2 ESP32-S3-WROOM-1, U3 AMS1117-3.3, U4 PCM5102A

Commit message: pcb編集中
Parts:
- removed the D1 at (167.2, 110.0)
- removed the D2 at (167.2, 112.6)
- removed the R2 at (170.0, 110.0)
- removed the R3 at (170.0, 112.5)
- C2, C5: footprint Capacitor_SMD:CP_Elec_5x5.9 -> Capacitor_SMD:C_0805_2012Metric
- C4: footprint Capacitor_SMD:CP_Elec_5x5.9 -> Capacitor_SMD:C_0603_1608Metric
- D2: renamed from D4; value LED -> Red LED
- J1: value USB_C_Receptacle_USB2.0_16P -> TYPE-C-31-M-12; footprint Connector_USB:USB_C_Receptacle_Amphenol_12401948E412A -> Connector_USB:USB_C_Receptacle_HRO_TYPE-C-31-M-12
- J11: value Conn_01x09 -> Conn_01x11; footprint Connector_PinHeader_2.54mm:PinHeader_1x09_P2.54mm_Vertical -> Connector_PinHeader_2.54mm:PinHeader_1x11_P2.54mm_Vertical
- SW1, SW2, SW3, SW4, SW5, SW6: value SW_Push -> TS-1187A-B-A-B; footprint Button_Switch_SMD:SW_Push_1P1T_NO_CK_KSC6xxG -> Button_Switch_SMD:SW_Push_1P1T_XKB_TS-1187A
- SW7: value SW_Wuerth_450301014042 -> SS-12D00-G3
- moved J2 211.4 mm to (20.5, 30.9), turned to 90 degrees
- moved C5 151.4 mm to (32.5, 50.5), turned to 180 degrees
- moved R4 144.6 mm to (32.5, 56.5)
- moved D2 143.7 mm to (36.0, 56.5)
- moved C4 132.5 mm to (36.0, 50.5)
- moved U3 128.4 mm to (34.0, 44.5)
- moved C2 125.7 mm to (32.5, 54.5)
- moved J11 122.5 mm to (104.3, 18.0), turned to 90 degrees
- moved SW7 119.2 mm to (65.1, 118.1)
- moved D1 119.2 mm to (103.5, 82.0)
- moved D3 119.2 mm to (103.5, 86.5)
- moved SW1 93.0 mm to (55.0, 30.0)
- moved J9 80.4 mm to (24.0, 10.5)
- moved U1 78.0 mm to (24.0, 50.0)
- moved C1 75.8 mm to (38.0, 19.9)
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- renumbered D3 to D1, D5 to D3, R4 to R2, R5 to R3, R6 to R4, R7 to R5, R8 to R6
Connections:
- C11 pad 1: +5V -> +3.3V
- C13 pad 1: +5V -> +3.3V
- C15 pad 1: +5V -> +3.3V
- C16 pad 1: +5V -> +3.3V
- C17 pad 1: +5V -> +3.3V
- C9 pad 1: +5V -> +3.3V
- J11 pad 8: +3.3V -> /IO45
- J11 pad 9: GND -> /IO46
- U4 pad 1: +5V -> +3.3V
- U4 pad 17: +5V -> +3.3V
- U4 pad 20: +5V -> +3.3V
- U4 pad 8: +5V -> +3.3V
Other:
- board outline removed

Commit message: 基板完成
Parts:
- removed SW5, SW6: TS-1187A-B-A-B, Button_Switch_SMD:SW_Push_1P1T_XKB_TS-1187A
- removed SW7: SS-12D00-G3, Button_Switch_THT:SW_Slide-03_Wuerth-WS-SLTV_10x2.5x6.4_P2.54mm
- added H1: MountingHole, MountingHole:MountingHole_3.2mm_M3, F.Cu at (24.0, 24.0)
- added H2: MountingHole, MountingHole:MountingHole_3.2mm_M3, F.Cu at (94.0, 24.0)
- added H3: MountingHole, MountingHole:MountingHole_3.2mm_M3, F.Cu at (24.0, 74.0)
- added H4: MountingHole, MountingHole:MountingHole_3.2mm_M3, F.Cu at (94.0, 74.0)
- added J12: Conn_01x02, Connector_JST:JST_XH_B2B-XH-A_1x02_P2.50mm_Vertical, F.Cu at (24.0, 52.0)
- added J13: Conn_01x04, Connector_PinHeader_2.54mm:PinHeader_1x04_P2.54mm_Vertical, F.Cu at (77.0, 43.0)
- J11: value Conn_01x11 -> Conn_01x04; footprint Connector_PinHeader_2.54mm:PinHeader_1x11_P2.54mm_Vertical -> Connector_PinHeader_2.54mm:PinHeader_1x04_P2.54mm_Vertical
- J2: footprint Connector_Audio:Jack_3.5mm_CUI_SJ-3523-SMT_Horizontal -> lcsc_footprints:C668608_PJ-313D
- J3, J4: value Conn_01x03 -> Conn_01x05; footprint Connector_PinHeader_2.54mm:PinHeader_1x03_P2.54mm_Vertical -> Connector_JST:JST_XH_B5B-XH-A_1x05_P2.50mm_Vertical
- J5: footprint Connector_PinHeader_2.54mm:PinHeader_1x03_P2.54mm_Vertical -> Connector_JST:JST_XH_B3B-XH-A_1x03_P2.50mm_Vertical
- J6, J7: footprint Connector_PinHeader_2.54mm:PinHeader_1x02_P2.54mm_Vertical -> Connector_JST:JST_XH_B2B-XH-A_1x02_P2.50mm_Vertical
- J8, J9: footprint Connector_PinHeader_2.54mm:PinHeader_1x05_P2.54mm_Vertical -> Connector_JST:JST_XH_B5B-XH-A_1x05_P2.50mm_Vertical
- moved J11 73.5 mm to (33.5, 37.5), turned to 0 degrees
- moved J8 60.5 mm to (86.0, 28.0), turned to -90 degrees
- moved D1 59.5 mm to (46.0, 66.5), turned to -90 degrees
- moved J2 44.6 mm to (35.0, 73.0), turned to 180 degrees
- moved SW3 43.3 mm to (69.0, 64.0)
- moved U3 42.8 mm to (65.0, 74.0), turned to 0 degrees
- moved J1 42.7 mm to (49.8, 75.5), turned to 0 degrees
- moved SW4 41.2 mm to (69.0, 34.0)
- moved C17 35.0 mm to (40.5, 62.1), turned to -90 degrees
- moved C4 34.6 mm to (59.4, 76.1), turned to 90 degrees
- moved C5 34.5 mm to (59.5, 72.0), turned to 90 degrees
- moved R3 34.4 mm to (51.5, 69.0), turned to -90 degrees
- moved R2 34.3 mm to (48.5, 69.0)
- moved D2 34.1 mm to (67.5, 69.5)
- moved C15 33.7 mm to (29.5, 59.6), turned to 90 degrees
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Connections:
- J11 pad 1: /IO3 -> /IO4
- J11 pad 2: /IO4 -> /IO18
- J11 pad 3: /IO18 -> /IO3
- J11 pad 4: /IO21 -> /IO46
- J3 pad 1: /ENC1_A -> +3.3V
- J3 pad 2: /ENC1_B -> /SW_MIC
- J3 pad 3: GND -> /ENC_B_MIC
- J4 pad 1: /ENC2_A -> +3.3V
- J4 pad 2: /ENC2_B -> /SW_SPK
- J4 pad 3: GND -> /ENC_B_SPK
- J5 pad 1: /ENC3_A -> /ENC_B_MOUSE
- J5 pad 2: /ENC3_B -> /ENC_A_MOUSE
- J6 pad 1: /SW_LEFT -> /SW_FORWARD
- J7 pad 1: /SW_RIGHT -> /SW_BACK
- SW3 pad 1: /SW3 -> /SW_LEFT
- SW4 pad 1: /SW4 -> /SW_RIGHT
- U2 pad 10: /SD_TX -> /BCLK_TX
- U2 pad 12: /SW7 -> /SW_SWAP
- U2 pad 17: /ENC1_A -> /ENC_A_MIC
- U2 pad 18: /ENC1_B -> /ENC_B_MIC
- U2 pad 19: /ENC2_A -> /SW_MIC
- U2 pad 20: /ENC2_B -> /ENC_A_SPK
- U2 pad 21: /ENC3_A -> /ENC_B_SPK
- U2 pad 22: /ENC3_B -> /SW_SPK
- U2 pad 24: /SW_LEFT -> /SW_FORWARD
- U2 pad 25: /SW_RIGHT -> /SW_BACK
- U2 pad 31: /SW3 -> /ENC_A_MOUSE
- U2 pad 32: /SW4 -> /ENC_B_MOUSE
- U2 pad 33: /SW5 -> /SW_LEFT
- U2 pad 34: /SW6 -> /SW_RIGHT
- U2 pad 8: /BCLK_TX -> /WS_TX
- U2 pad 9: /WS_TX -> /SD_TX
Routing:
- net +3.3V: track 0.00 -> 189.4 mm, vias 0 -> 1
- net Net-(D3-A): track 0.00 -> 61.9 mm
- net /SW_LEFT: track 0.00 -> 36.1 mm, vias 0 -> 2
- net +5V: track 0.00 -> 34.1 mm
- net GND: track 0.00 -> 34.0 mm, vias 0 -> 135
- net /EN: track 0.00 -> 31.5 mm, vias 0 -> 3
- net /SW_BACK: track 0.00 -> 30.4 mm
- net /SW_SWAP: track 0.00 -> 28.1 mm, vias 0 -> 2
- net /ENC_A_MOUSE: track 0.00 -> 25.7 mm
- net /ENC_B_MOUSE: track 0.00 -> 25.2 mm
- net /USB_DM: track 0.00 -> 25.1 mm, vias 0 -> 2
- net /WS_TX: track 0.00 -> 25.0 mm
- net /SD_RX: track 0.00 -> 24.2 mm
- net /JOY_SW: track 0.00 -> 23.8 mm
- net /SD_TX: track 0.00 -> 23.8 mm
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- added copper zone on B.Cu, net GND
- added copper zone on F.Cu, net GND
Other:
- board outline added: 78 x 58 mm

Commit message: 基板発注前更新
Parts:
- SW3, SW4: value TS-1187A-B-A-B -> Tactile Switch 6x6x6mm THT; footprint Button_Switch_SMD:SW_Push_1P1T_XKB_TS-1187A -> Button_Switch_THT:SW_PUSH_6mm
- moved J9 63.9 mm to (87.0, 24.0), turned to 180 degrees
- moved D3 58.9 mm to (22.5, 46.5), turned to -90 degrees
- moved J1 55.1 mm to (35.0, 22.5), turned to 180 degrees
- moved R1 51.4 mm to (94.5, 39.5), turned to 180 degrees
- moved J2 50.3 mm to (50.0, 25.0), turned to 0 degrees
- moved C1 49.0 mm to (92.4, 39.5), turned to 180 degrees
- moved C4 48.2 mm to (26.4, 40.9), turned to 0 degrees
- moved J8 47.0 mm to (87.5, 75.0), turned to 180 degrees
- moved C6 46.8 mm to (59.2, 22.9), turned to -90 degrees
- moved C10 46.5 mm to (73.3, 23.4), turned to 90 degrees
- moved C14 46.1 mm to (71.8, 23.4), turned to 90 degrees
- moved C9 45.7 mm to (70.3, 23.3), turned to -90 degrees
- moved U3 45.7 mm to (28.5, 46.5), turned to -90 degrees
- moved C13 45.5 mm to (68.8, 23.4), turned to -90 degrees
- moved C15 45.1 mm to (63.5, 30.0), turned to 0 degrees
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Connections:
- J11 pad 3: /IO3 -> /IO46
- J11 pad 4: /IO46 -> /IO3
- J9 pad 1: /BCLK_RX -> +3.3V
- J9 pad 2: /WS_RX -> GND
- J9 pad 3: /SD_RX -> /BCLK_RX
- J9 pad 4: +3.3V -> /WS_RX
- J9 pad 5: GND -> /SD_RX
- U1 pad 1: /USB_DM -> Net-(J1-D--PadA7)
- U1 pad 3: /USB_DP -> Net-(J1-D+-PadA6)
- U1 pad 4: Net-(J1-D+-PadA6) -> /USB_DP
- U1 pad 6: Net-(J1-D--PadA7) -> /USB_DM
Routing:
- net /SW_SPK: track 12.5 -> 47.0 mm
- net Net-(D3-A): track 61.9 -> 94.8 mm
- net /ENC_B_SPK: track 15.6 -> 46.5 mm
- net /SW_MIC: track 11.2 -> 41.6 mm
- net GND: track 34.0 -> 4.49 mm, vias 135 -> 77
- net /ENC_A_SPK: track 18.6 -> 46.0 mm
- net /ENC_B_MIC: track 14.2 -> 41.1 mm
- net /USB_DP: track 23.0 -> 49.1 mm, vias 2 -> 0
- net /USB_DM: track 25.1 -> 48.8 mm, vias 2 -> 0
- net /SW_RIGHT: track 13.3 -> 36.6 mm
- net /ENC_A_MIC: track 17.3 -> 40.5 mm
- net /SW_FORWARD: track 22.6 -> 36.5 mm
- net /SW_LEFT: track 36.1 -> 25.5 mm
- net /EN: track 31.5 -> 21.1 mm, vias 3 -> 2
- net +5V: track 34.1 -> 26.3 mm
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
Commit message: 配置エラー修正
Parts:
- moved J5 14.0 mm to (59.5, 67.0)
- moved SW3 5.50 mm to (71.2, 66.2)
- moved SW4 0.50 mm to (71.2, 31.2)
Routing:
- net /ENC_B_MOUSE: track 25.5 -> 31.9 mm
- net /ENC_A_MOUSE: track 27.0 -> 32.2 mm
- net /SW_LEFT: track 25.5 -> 26.3 mm
- net /SW_RIGHT: track 36.6 -> 36.9 mm, vias 2 -> 1
